File: v2.0/output/pcbs/left.kicad_pcb (KiCad board)
At the start: 2 copper layers, 121.8 x 95.7 mm, 52 parts

Commit message: feature: finish left hand-side
Parts:
- removed D22, D23, D24: , ComboDiode
- removed S22, S23, S24: , MX
- moved T1 236.0 mm to (83.2, -59.0), turned to 0 degrees
- moved S9 224.6 mm to (38.0, -46.0)
- moved D9 220.9 mm to (29.5, -41.5)
- moved D21 220.7 mm to (91.5, -39.0)
- moved B1 219.9 mm to (105.0, -58.0), turned to 0 degrees
- moved S17 218.7 mm to (95.0, -43.0)
- moved S21 206.4 mm to (95.0, -24.0), turned to -180 degrees
- moved S5 205.9 mm to (19.0, -19.0)
- moved S6 205.3 mm to (19.0, -38.0)
- moved D5 202.3 mm to (10.5, -14.5)
- moved D6 201.8 mm to (10.5, -33.5)
- moved JST1 193.9 mm to (73.0, -52.0)
- moved S1 187.2 mm to (0.00, 0.00)
- moved S2 186.7 mm to (0.00, -19.0)
- moved S3 186.2 mm to (0.00, -38.0)
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Connections:
- net middle_bottom renamed ColE_Row1
- net middle_home renamed ColE_Row2
- net middle_num renamed ColF_Row1
- net middle_top renamed ColE_Row3
- net outer_bottom renamed ColA_Row1
- net outer_home renamed ColA_Row2
- net outer_num renamed ColB_Row1
- net outer_top renamed ColA_Row3
- net pinky_bottom renamed ColB_Row2
- net pinky_home renamed ColB_Row3
- net pinky_num renamed ColC_Row2
- net pinky_top renamed ColC_Row1
- net ring_bottom renamed ColC_Row3
- net ring_home renamed ColD_Row1
- net ring_num renamed ColD_Row3
- net ring_top renamed ColD_Row2
- D1 pad 1: P100 -> P011
- D10 pad 1: P024 -> P011
- D11 pad 1: P022 -> P009
- D12 pad 1: P020 -> P100
- D13 pad 1: P100 -> P011
- D14 pad 1: P024 -> P009
- D15 pad 1: P022 -> P100
- D16 pad 1: P020 -> P011
- D17 pad 1: P100 -> P115
- D17 pad 2: index_bottom -> ColD_Row0
- D18 pad 1: P024 -> P115
- D18 pad 2: index_home -> ColE_Row0
- D19 pad 1: P022 -> P115
- D19 pad 2: index_top -> ColF_Row0
- D2 pad 1: P024 -> P009
- D20 pad 1: P020 -> P009
- D20 pad 2: index_num -> ColF_Row2
- D21 pad 2: inner_bottom -> ColF_Row3
- D3 pad 1: P022 -> P100
- D4 pad 1: P020 -> P011
- D5 pad 1: P100 -> P009
- D6 pad 1: P024 -> P100
- D7 pad 1: P022 -> P011
- D8 pad 1: P020 -> P009
- S1 pad 1: P106 -> P006
- S10 pad 1: P011 -> P020
- S11 pad 1: P011 -> P020
- S12 pad 1: P011 -> P020
- S13 pad 1: P006 -> P022
- S14 pad 1: P006 -> P022
- S15 pad 1: P006 -> P022
- S16 pad 1: P006 -> P029
- S17 pad 1: P008 -> P029
- S17 pad 2: index_bottom -> ColF_Row3
- S18 pad 1: P008 -> P020
- S18 pad 2: index_home -> ColD_Row0
- S19 pad 1: P008 -> P022
- S19 pad 2: index_top -> ColE_Row0
- S2 pad 1: P106 -> P006
- S20 pad 1: P008 -> P029
- S20 pad 2: index_num -> ColF_Row0
- S21 pad 1: P031 -> P029
- S21 pad 2: inner_bottom -> ColF_Row2
- S3 pad 1: P106 -> P006
- S4 pad 1: P106 -> P008
- S5 pad 1: P104 -> P008
- S6 pad 1: P104 -> P008
- S7 pad 1: P104 -> P017
- S8 pad 1: P104 -> P017
- S9 pad 1: P011 -> P017
Routing:
- net P104: track 152.4 -> 0.00 mm, vias 1 -> 0
- net P020: track 146.5 -> 0.00 mm
- net P006: track 106.6 -> 0.00 mm, vias 1 -> 0
- net P031: track 96.0 -> 0.00 mm
- net P008: track 85.0 -> 0.00 mm, vias 1 -> 0
- net P011: track 80.0 -> 0.00 mm
- net P106: track 80.0 -> 0.00 mm
- net inner_num: track 43.7 -> 0.00 mm
- net ColF_Row1: track 24.1 -> 0.00 mm
- net ColD_Row3: track 24.0 -> 0.00 mm
- net ColC_Row2: track 23.3 -> 0.00 mm
- net ColB_Row1: track 23.3 -> 0.00 mm
- net index_num: track 23.1 -> 0.00 mm
- net ColA_Row3: track 21.8 -> 0.00 mm
Other:
- board size 121.8 x 95.7 mm -> 147.4 x 109 mm
- net class Default added: clearance 0.2, trace_width 0.25, via_dia 0.8, via_drill 0.4
- board text added: "KiwiBoard Rev1"
- board text removed: "KIWI.BOARD"
