File: v2.0/output/pcbs/rev1/left.kicad_pcb (KiCad board)
At the start: 2 copper layers, 140.3 x 101 mm, 46 parts

Commit message: feature: complete v2.0. Ready for pre-prod
Routing:
- net ColD_Row1: track 24.4 -> 22.9 mm
- net ColC_Row2: track 24.6 -> 23.3 mm
- net ColD_Row2: track 24.4 -> 23.2 mm
- net ColE_Row2: track 23.3 -> 22.1 mm
- net ColA_Row3: track 23.0 -> 21.8 mm
- net ColE_Row1: track 22.6 -> 21.5 mm
- net ColC_Row1: track 23.0 -> 21.9 mm
- net ColB_Row1: track 23.0 -> 21.9 mm
- net ColA_Row1: track 23.0 -> 21.9 mm
- net ColF_Row0: track 22.9 -> 21.9 mm
- net ColB_Row3: track 23.0 -> 22.0 mm
- net ColC_Row3: track 23.0 -> 22.0 mm
- net ColD_Row0: track 23.9 -> 22.9 mm
- net ColA_Row2: track 23.0 -> 22.0 mm
- net ColF_Row1: track 23.7 -> 22.8 mm
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